File: hardware/kicad/DrunkPCDebugger.kicad_sch (KiCad schematic)
At the start: 92 parts, among them Q1 2N7002K-T1-GE3, Q2 AO3401A, Q3 AO3401A, SW2 TS3643TP, SW3 TS3643TP, U1 74LVX4245MTCX, U10 A-SC6302R6AGHC-A03-2T, U2 STM32H723VGT6, U3 74LVX4245MTCX, U4 74LVX4245MTCX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

Commit message: Fab
Parts:
- added 5v_1: 5v, TestPoint:TestPoint_Pad_D1.5mm, symbol Connector:TestPoint
- added 5v_bus_1: 5vBus, TestPoint:TestPoint_Pad_D1.5mm, symbol Connector:TestPoint
Connections:
- net USB_VBUS is gone; now on net +5V: C38.1, C39.2, U6.3 (VIN), USB1.A4B9 (VBUS), USB1.B4A9 (VBUS)
- net +5V: now also 5v_1.1
- net BUS_5V: now also 5v_bus_1.1
