File: hardware/kicad/DrunkPCDebugger.kicad_sch (KiCad schematic)
At the start: 96 parts, among them Q1 2N7002K-T1-GE3, Q2 AO3401A, Q3 AO3401A, SW2 TS3643TP, SW3 TS3643TP, U1 74LVX4245MTCX, U10 A-SC6302R6AGHC-A03-2T, U2 STM32H723VGT6, U3 74LVX4245MTCX, U4 74LVX4245MTCX, U5 X6521FV-2X27-C85D32, U6 AMS1117-3_3, U7 74LVX4245MTCX, U8 SN74LVC3G17DCTR, U9 SN74AHCT125DR, X1 X322525MOB4SI

Commit message: Fix errata in rev 2.
Connections:
- net MCU_CTRL_BUS_DIR: now also U2.25 (PA3); no longer U2.9 (PC15-OSC32_OUT)
Changed lines of the file:
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@@
 	)
 	(no_connect
-		(at 137.16 96.52)
-	)
-	(no_connect
 		(at 137.16 132.08)
 	)
@@
 	)
 	(no_connect
+		(at 137.16 55.88)
+	)
+	(no_connect
 		(at 137.16 71.12)
 	)
@@
 	(wire
 		(pts
-			(xy 114.3 50.8) (xy 133.35 50.8)
-		)
-		(stroke
-			(width 0)
-			(type default)
-		)
-	)
-	(wire
-		(pts
 			(xy 274.32 24.13) (xy 274.32 52.07)
 		)
@@
 	(wire
 		(pts
-			(xy 133.35 50.8) (xy 133.35 55.88)
-		)
-		(stroke
-			(width 0)
-			(type default)
-		)
-	)
-	(wire
-		(pts
 			(xy 77.47 205.74) (xy 71.12 205.74)
 		)
@@
 	(wire
 		(pts
-			(xy 133.35 55.88) (xy 137.16 55.88)
-		)
-		(stroke
-			(width 0)
-			(type default)
-		)
-	)
-	(wire
-		(pts
 			(xy 180.34 40.64) (xy 177.8 40.64)
 		)
@@
 	(wire
 		(pts
+			(xy 121.92 96.52) (xy 137.16 96.52)
+		)
+		(stroke
+			(width 0)
+			(type default)
+		)
+	)
+	(wire
+		(pts
 			(xy 238.76 52.07) (xy 251.46 52.07)
 		)
@@
 		)
 	)
-	(label "MCU_CTRL_BUS_DIR"
-		(at 114.3 50.8 180)
-		(effects
-			(font
-				(size 1.27 1.27)
-			)
-			(justify right bottom)
-		)
-	)
 	(label "MCU_A0"
 		(at 186.69 83.82 0)
@@
 		(effects
 			(font
+				(size 1.27 1.27)
+			)
+			(justify right bottom)
+		)
+	)
+	(label "MCU_CTRL_BUS_DIR"
+		(at 121.92 96.52 180)
+		(effects
+			(font

Commit message: Replace components
Parts:
- C59, C60, C61, C62, C63, C64, C65, C66, C67, C68, C69, C70, C71, C72, C73, C74: value CL10B104KB8NNNC -> CC0603KRX7R9BB104; symbol JLCImport:CL10B104KB8NNNC -> JLCImport:CC0603KRX7R9BB104; LCSC C1591 -> C14663; Manufacturer Samsung Electro-Mechanics -> YAGEO; Manufacturer Part CL10B104KB8NNNC -> CC0603KRX7R9BB104
- R1, R10, R11, R12, R13, R14, R15, R16, R17, R18, R19, R2, R20, R21, R22, R23, R24, R3, R30, R36, R37, R38, R39, R4, R40, R41, R5, R6, R7, R8, R9: value RT0603BRD07100RL -> 0603WAF1000T5E; symbol JLCImport:RT0603BRD07100RL -> JLCImport:0603WAF1000T5E; LCSC C122970 -> C22775; Manufacturer YAGEO -> UNI-ROYAL(Uniroyal Elec); Manufacturer Part RT0603BRD07100RL -> 0603WAF1000T5E
- R25, R26: value FRC0603F5101TS -> 0603WAF5101T5E; symbol JLCImport:FRC0603F5101TS -> JLCImport:0603WAF5101T5E; LCSC C2907044 -> C23186; Manufacturer FOJAN -> UNI-ROYAL(Uniroyal Elec); Manufacturer Part FRC0603F5101TS -> 0603WAF5101T5E
- R27, R28, R31: value FRC0603F1001TS -> 0603WAF1001T5E; symbol JLCImport:FRC0603F1001TS -> JLCImport:0603WAF1001T5E; LCSC C2907002 -> C21190; Manufacturer FOJAN -> UNI-ROYAL(Uniroyal Elec); Manufacturer Part FRC0603F1001TS -> 0603WAF1001T5E
- R29: value FRC0603J104_TS -> 0603WAF1003T5E; symbol JLCImport:FRC0603J104_TS -> JLCImport:0603WAF1003T5E; LCSC C2907088 -> C25803; Manufacturer FOJAN -> UNI-ROYAL(Uniroyal Elec); Manufacturer Part FRC0603J104 TS -> 0603WAF1003T5E
- R42, R43, R47, R48, R49, R52, R53, R54, R55, R56: value RT0603BRD0710KL -> 0603WAF1002T5E; symbol JLCImport:RT0603BRD0710KL -> JLCImport:0603WAF1002T5E; LCSC C95204 -> C25804; Manufacturer YAGEO -> UNI-ROYAL(Uniroyal Elec); Manufacturer Part RT0603BRD0710KL -> 0603WAF1002T5E

Commit message: Replace parts
Parts:
- removed C3, C4: GRM21BR71A225KA01L, Capacitor_SMD:C_0805_2012Metric, symbol JLCImport:GRM21BR71A225KA01L
- removed C39: GCM21BR71A106KE22L, JLCImport:GCM21BR71A106KE22L, symbol JLCImport:GCM21BR71A106KE22L
- removed C5, C6: CC0603KRX7R0BB103, Capacitor_SMD:C_0603_1608Metric, symbol JLCImport:CC0603KRX7R0BB103
- removed C9: 25TQC22MYFB, JLCImport:25TQC22MYFB, symbol JLCImport:25TQC22MYFB
- added C3: 100uF 6.3V, Capacitor_Tantalum_SMD:CP_EIA-3528-21_Kemet-B, symbol JLCImport:TAJB107K006RNJ
- added C4: 10uF 25V, Capacitor_SMD:C_0805_2012Metric, symbol JLCImport:CL21A106KAYNNNE
- added C5, C6: 2.2uF 16V, Capacitor_SMD:C_0603_1608Metric, symbol JLCImport:CL10A225KO8NNNC
- added C75, C76: CC0603KRX7R9BB104, Capacitor_SMD:C_0603_1608Metric, symbol JLCImport:CC0603KRX7R9BB104
Connections:
- net +3V3: now also C3.1
- net +5V: now also C4.1
- net GND: now also C3.2, C4.2, C5.2, C6.2, C75.1, C76.1
- net MCU_BOOT0: now also C76.2
- net MCU_RESET: now also C75.2
- net MCU_VCAP: now also C5.1, C6.1

Commit message: Replace components
Parts:
- removed H2: PZ254R-11-04P, JLCImport:PZ254R-11-04P, symbol JLCImport:PZ254R-11-04P
- removed Q1: 2N7002K-T1-GE3, JLCImport:2N7002K-T1-GE3, symbol JLCImport:2N7002K-T1-GE3
- removed U9: SN74AHCT125DR, JLCImport:SN74AHCT125DR, symbol JLCImport:SN74AHCT125DR
- added D1: USBLC6-2SC6_C2687116, JLCImport:USBLC6-2SC6_C2687116, symbol JLCImport:USBLC6-2SC6_C2687116
- added H2: PZ254R-11-05P, JLCImport:PZ254R-11-05P, symbol JLCImport:PZ254R-11-05P
- added Q4: AO3400A, JLCImport:AO3400A, symbol JLCImport:AO3400A
- added R44: 0603WAF1000T5E, Resistor_SMD:R_0603_1608Metric, symbol JLCImport:0603WAF1000T5E
- added U11: SN74LVC3G07DCTR, JLCImport:SN74LVC3G07DCTR, symbol JLCImport:SN74LVC3G07DCTR
- U1, U3, U4, U7: value 74LVX4245MTCX -> SN74LVC4245APWR; footprint JLCImport:74LVX4245MTCX -> JLCImport:SN74LVC4245APWR; symbol JLCImport:74LVX4245MTCX -> JLCImport:SN74LVC4245APWR; LCSC C61186 -> C7859; Manufacturer onsemi -> Texas Instruments; Manufacturer Part 74LVX4245MTCX -> SN74LVC4245APWR
Connections:
- net +3V3: now also C66.1, R47.1, R48.1, R49.1, R54.2, U11.8 (VCC)
- net +5V: now also Q3.3 (D), D1.5 (VBUS), H2.1; no longer C66.1, Q3.2 (S), R29.1, R54.2
- net BUS_5V: now also Q2.3 (D); no longer Q2.2 (S)
- net BUS_BUSREQ/: now also U11.2 (3Y)
- net BUS_RES/: now also R44.2
- net BUS_WAIT/: now also U11.7 (1Y)
- net GND: now also D1.2 (GND), H2.5, Q4.2 (S), U11.4 (GND); no longer R47.1, R48.1, R49.1
- net MCU_BUSREQ/: now also U11.6 (3A)
- net MCU_RESET: now also H2.4
- net MCU_USB_DM: now also D1.1 (I/O1); no longer USB1.A7 (Dn1), USB1.B7 (Dn2)
- net MCU_USB_DP: now also D1.3 (I/O2); no longer USB1.A6 (Dp1), USB1.B6 (Dp2)
- net MCU_WAIT/: now also U11.1 (1A)
- net MCU_Z80_RES/: now also U11.3 (2A)
- net SWCLK: now also H2.3
- net SWDIO: now also H2.2
- net at R31.2, R55.2: now also Q4.1 (G)
- net at R30.2: now also Q4.3 (D)
- net at Q2.1 (G), Q3.1 (G), R30.1: now also R29.1; no longer R29.2
- new net: R44.1, U11.5 (2Y)
- new net: D1.4 (I/O2), USB1.A6 (Dp1), USB1.B6 (Dp2)
- new net: D1.6 (I/O1), USB1.A7 (Dn1), USB1.B7 (Dn2)
- new net: Q2.2 (S), Q3.2 (S), R29.2
- no-connect marks 41 -> 40
Other:
- moved on the sheet: Q2, Q3, R52, R53, R54

Commit message: Fixes
Parts:
- removed R29: 0603WAF1003T5E, Resistor_SMD:R_0603_1608Metric, symbol JLCImport:0603WAF1003T5E
- removed R30: 0603WAF1000T5E, Resistor_SMD:R_0603_1608Metric, symbol JLCImport:0603WAF1000T5E
- added C7: 2.2uF, Capacitor_SMD:C_0603_1608Metric, symbol JLCImport:CL10A225KO8NNNC
- added Q1: AO3400A, JLCImport:AO3400A, symbol JLCImport:AO3400A
- added R32: 0603WAF1001T5E, Resistor_SMD:R_0603_1608Metric, symbol JLCImport:0603WAF1001T5E
- added R33: 0603WAF1003T5E, Resistor_SMD:R_0603_1608Metric, symbol JLCImport:0603WAF1003T5E
- added R34, R35: 47kΩ, Resistor_SMD:R_0603_1608Metric, symbol JLCImport:0603WAF4702T5E
- added R57, R58: 0603WAF1002T5E, Resistor_SMD:R_0603_1608Metric, symbol JLCImport:0603WAF1002T5E
- U2: value STM32H723VGT6 -> STM32H723VET6; footprint JLCImport:STM32H723VGT6 -> JLCImport:STM32H723VET6; symbol JLCImport:STM32H723VGT6 -> JLCImport:STM32H723VET6; LCSC C730142 -> C730141; Manufacturer Part STM32H723VGT6 -> STM32H723VET6
Connections:
- net +3V3: now also H2.1; no longer R56.1
- net +5V: no longer C67.1, C69.1, C71.1, C73.1, H2.1, U1.1 (VCCA), U3.1 (VCCA), U4.1 (VCCA), U7.1 (VCCA)
- net BUS_5V: now also C67.1, C69.1, C71.1, C73.1, R56.1, U1.1 (VCCA), U3.1 (VCCA), U4.1 (VCCA), U7.1 (VCCA), R34.2
- net GND: now also Q1.2 (S), R33.1, R57.2
- net MCU_BUS_OE/: now also R32.1; no longer R56.2, U1.22 (OE#), U3.22 (OE#), U4.22 (OE#), U7.22 (OE#)
- net MCU_BUS_5V_ADC: now reaches U2.67 (PA8)
- net MCU_BUS_5V_ADC: now also R33.2, R34.1
- net at Q2.1 (G), Q3.1 (G): now also C7.1, R35.2, R58.2
- net at Q4.3 (D): now also R58.1
- net at Q2.2 (S), Q3.2 (S): now also C7.2, R35.1
- new net: Q1.1 (G), R32.2, R57.1
- new net BUS_OE/: Q1.3 (D), R56.2, U1.22 (OE#), U3.22 (OE#), U4.22 (OE#), U7.22 (OE#)
- no-connect marks 40 -> 39

Commit message: Pcb production
Parts:
- added R29, R30, R45, R46: 10kΩ, Resistor_SMD:R_0603_1608Metric, symbol JLCImport:0603WAF1002T5E
Connections:
- net GND: now also R29.1, R30.1, R45.1, R46.1
- net at U7.10 (A8): now also R30.2
- net at U7.14 (B8): now also R46.2
- net at U7.21 (B1): now also R45.2
- net at U7.3 (A1): now also R29.2
- no-connect marks 39 -> 35
Other:
- moved on the sheet: C69, C70
