File: hardware/kicad/DrunkPCDebugger.kicad_pcb (KiCad board)
At the start: 4 copper layers, 71 x 57.5 mm, 94 parts, among them Q1 2N7002K-T1-GE3, Q2 AO3401A, Q3 AO3401A, SW2 TS3643TP, SW3 TS3643TP, U1 74LVX4245MTCX, U10 A-SC6302R6AGHC-A03-2T, U2 STM32H723VGT6, U3 74LVX4245MTCX, U4 74LVX4245MTCX, U5 X6521FV-2X27-C85D32, U6 AMS1117-3_3, U7 74LVX4245MTCX, U8 SN74LVC3G17DCTR, U9 SN74AHCT125DR, X1 X322525MOB4SI

Commit message: stm, fix
Other:
- board text added: "30.06.2026, Earth, Milky Way"
- board text removed: "30.06.2026, Moscow, Russia"
