File: hardware/kicad/DrunkPCDebugger.kicad_pcb (KiCad board)
At the start: 4 copper layers, 71 x 57.5 mm, 96 parts, among them Q1 2N7002K-T1-GE3, Q2 AO3401A, Q3 AO3401A, SW2 TS3643TP, SW3 TS3643TP, U1 74LVX4245MTCX, U10 A-SC6302R6AGHC-A03-2T, U2 STM32H723VGT6, U3 74LVX4245MTCX, U4 74LVX4245MTCX, U5 X6521FV-2X27-C85D32, U6 AMS1117-3_3, U7 74LVX4245MTCX, U8 SN74LVC3G17DCTR, U9 SN74AHCT125DR, X1 X322525MOB4SI

Commit message: Fix errata in rev 2.
Connections:
- U2 pad 25: unconnected-(U2-PA3-Pad25) -> /MCU_CTRL_BUS_DIR
- U2 pad 9: /MCU_CTRL_BUS_DIR -> unconnected-(U2-PC15-OSC32_OUT-Pad9)
Routing:
- net /MCU_CTRL_BUS_DIR: track 33.8 -> 42.6 mm
Changed lines of the file:
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@@
 			(size 0.3 1.6)
 			(layers "F.Cu" "F.Mask" "F.Paste")
-			(net "/MCU_CTRL_BUS_DIR")
+			(net "unconnected-(U2-PC15-OSC32_OUT-Pad9)")
 			(pinfunction "PC15-OSC32_OUT_9")
-			(pintype "unspecified")
+			(pintype "unspecified+no_connect")
 		)
 		(pad "10" smd oval
@@
 			(size 0.3 1.6)
 			(layers "F.Cu" "F.Mask" "F.Paste")
-			(net "unconnected-(U2-PA3-Pad25)")
+			(net "/MCU_CTRL_BUS_DIR")
 			(pinfunction "PA3_25")
-			(pintype "unspecified+no_connect")
+			(pintype "unspecified")
 		)
 		(pad "26" smd oval
@@
 	)
 	(segment
-		(start 90.95 60.15)
-		(end 90.85 60.25)
+		(start 91.15 52.25)
+		(end 91.2 52.2)
 		(width 0.2)
 		(layer "F.Cu")
@@
 	)
 	(segment
-		(start 95.925 77)
-		(end 96.1 76.825)
+		(start 89.50175 52.25)
+		(end 91.15 52.25)
 		(width 0.2)
 		(layer "F.Cu")
@@
 	)
 	(segment
-		(start 95.925 77.6)
-		(end 95.925 77)
+		(start 95.925 77)
+		(end 96.1 76.825)
 		(width 0.2)
 		(layer "F.Cu")
@@
 	)
 	(segment
-		(start 90.85 60.25)
-		(end 89.50175 60.25)
+		(start 95.925 77.6)
+		(end 95.925 77)
 		(width 0.2)
 		(layer "F.Cu")
@@
 	)
 	(via
-		(at 90.95 60.15)
+		(at 96.95 83.575)
 		(size 0.6)
 		(drill 0.3)
@@
 	)
 	(via
-		(at 96.95 83.575)
+		(at 91.2 52.2)
 		(size 0.6)
 		(drill 0.3)
@@
 	)
 	(segment
+		(start 95.575 60.825)
+		(end 94.8 60.05)
+		(width 0.2)
+		(layer "B.Cu")
+		(net "/MCU_CTRL_BUS_DIR")
+	)
+	(segment
+		(start 94.8 60.05)
+		(end 92.225 60.05)
+		(width 0.2)
+		(layer "B.Cu")
+		(net "/MCU_CTRL_BUS_DIR")
+	)
+	(segment
 		(start 95.9 75.175)
 		(end 96.1 75.375)
@@
 	)
 	(segment
-		(start 97.025 71.537648)
-		(end 95.9 72.662648)
+		(start 95.575 62.3)
+		(end 95.575 60.825)
 		(width 0.2)
 		(layer "B.Cu")
@@
 	)
 	(segment
-		(start 95.575 62.3)
-		(end 94.225 63.65)
+		(start 97.025 71.537648)
+		(end 95.9 72.662648)
 		(width 0.2)
 		(layer "B.Cu")
@@
 	)
 	(segment
-		(start 95.575 60.825)
+		(start 90.4 53)
+		(end 91.2 52.2)
+		(width 0.2)
+		(layer "B.Cu")
+		(net "/MCU_CTRL_BUS_DIR")
+	)
+	(segment
+		(start 94.225 63.65)
 		(end 95.575 62.3)
 		(width 0.2)
@@
 	)
 	(segment
-		(start 94.9 60.15)
-		(end 95.575 60.825)
+		(start 90.4 59.8)
+		(end 90.4 53)
 		(width 0.2)
 		(layer "B.Cu")
@@
 	)
 	(segment
-		(start 90.95 60.15)
-		(end 94.9 60.15)
+		(start 92.225 60.05)
+		(end 90.65 60.05)
+		(width 0.2)
+		(layer "B.Cu")
+		(net "/MCU_CTRL_BUS_DIR")
+	)
+	(segment
+		(start 90.65 60.05)
+		(end 90.4 59.8)
 		(width 0.2)
 		(layer "B.Cu")

Commit message: Fix silk
Parts:
- moved R27 12.3 mm to (87.0, 48.0)
- moved R28 12.3 mm to (85.3, 48.0)
- moved 5v_bus_1 0.50 mm to (105.0, 74.3)
- moved 3v3_1 0.30 mm to (100.0, 74.3)
- moved 5v_1 0.10 mm to (110.0, 74.3)
Routing:
- net Net-(R28-Pad1): track 4.45 -> 15.2 mm
- net Net-(R27-Pad2): track 4.37 -> 15.1 mm
- net /MCU_LED: track 12.4 -> 15.0 mm
Other:
- board text removed: "STM32H723VGT6"

Commit message: Replace components
Parts:
- C59, C60, C61, C62, C63, C64, C65, C66, C67, C68, C69, C70, C71, C72, C73, C74: value CL10B104KB8NNNC -> CC0603KRX7R9BB104
- R1, R10, R11, R12, R13, R14, R15, R16, R17, R18, R19, R2, R20, R21, R22, R23, R24, R3, R30, R36, R37, R38, R39, R4, R40, R41, R5, R6, R7, R8, R9: value RT0603BRD07100RL -> 0603WAF1000T5E
- R25, R26: value FRC0603F5101TS -> 0603WAF5101T5E
- R27, R28, R31: value FRC0603F1001TS -> 0603WAF1001T5E
- R29: value FRC0603J104_TS -> 0603WAF1003T5E
- R42, R43, R47, R48, R49, R52, R53, R54, R55, R56: value RT0603BRD0710KL -> 0603WAF1002T5E

Commit message: Replace parts
Parts:
- removed C39: GCM21BR71A106KE22L, JLCImport:GCM21BR71A106KE22L
- removed C9: 25TQC22MYFB, JLCImport:25TQC22MYFB
- added C75: CC0603KRX7R9BB104, Capacitor_SMD:C_0603_1608Metric, B.Cu at (55.4, 52.0)
- added C76: CC0603KRX7R9BB104, Capacitor_SMD:C_0603_1608Metric, B.Cu at (55.2, 62.5)
- C3: value GRM21BR71A225KA01L -> 100uF 6.3V; footprint Capacitor_SMD:C_0805_2012Metric -> Capacitor_Tantalum_SMD:CP_EIA-3528-21_Kemet-B; moved to B.Cu
- C4: value GRM21BR71A225KA01L -> 10uF 25V; moved to B.Cu
- C5, C6: value CC0603KRX7R0BB103 -> 2.2uF 16V; moved to F.Cu
- moved C4 40.8 mm to (111.3, 64.8), turned to -90 degrees
- moved C3 30.8 mm to (101.3, 65.9), turned to 90 degrees
- moved C6 24.9 mm to (75.7, 48.4), turned to 180 degrees
- moved C5 18.8 mm to (70.5, 63.2)
Connections:
- C3 pad 1: GND -> +3V3
- C3 pad 2: /MCU_VCAP -> GND
- C4 pad 1: /MCU_VCAP -> +5V
- C5 pad 1: /MCU_RESET -> /MCU_VCAP
- C6 pad 1: /MCU_BOOT0 -> /MCU_VCAP
Routing:
- net /MCU_VCAP: track 35.1 -> 34.2 mm, vias 4 -> 2

Commit message: Replace components
Parts:
- removed Q1: 2N7002K-T1-GE3, JLCImport:2N7002K-T1-GE3
- removed U9: SN74AHCT125DR, JLCImport:SN74AHCT125DR
- added D1: USBLC6-2SC6_C2687116, JLCImport:USBLC6-2SC6_C2687116, B.Cu at (70.2, 47.0)
- added Q4: AO3400A, JLCImport:AO3400A, F.Cu at (113.0, 75.1)
- added R44: 0603WAF1000T5E, Resistor_SMD:R_0603_1608Metric, F.Cu at (88.1, 72.0)
- added U11: SN74LVC3G07DCTR, JLCImport:SN74LVC3G07DCTR, F.Cu at (84.4, 74.1)
- H2: value PZ254R-11-04P -> PZ254R-11-05P; footprint JLCImport:PZ254R-11-04P -> JLCImport:PZ254R-11-05P
- U1, U3, U4, U7: value 74LVX4245MTCX -> SN74LVC4245APWR; footprint JLCImport:74LVX4245MTCX -> JLCImport:SN74LVC4245APWR
- moved R29 2.72 mm to (115.5, 81.5), turned to -90 degrees
- moved C66 2.10 mm to (81.1, 73.0), turned to 0 degrees
- moved H2 1.28 mm to (108.8, 56.2)
- moved Q2 1.03 mm to (110.4, 82.9), turned to 0 degrees
- moved Q3 0.42 mm to (113.0, 79.6), turned to -90 degrees
Connections:
- C66 pad 1: +5V -> +3V3
- H2 pad 4: GND -> /MCU_RESET
- Q2 pad 2: BUS_5V -> Net-(Q2-S)
- Q2 pad 3: Net-(Q2-D) -> BUS_5V
- Q3 pad 2: +5V -> Net-(Q2-S)
- Q3 pad 3: Net-(Q2-D) -> +5V
- R29 pad 1: +5V -> Net-(Q2-G)
- R29 pad 2: Net-(Q2-G) -> Net-(Q2-S)
- R47 pad 1: GND -> +3V3
- R48 pad 1: GND -> +3V3
- R49 pad 1: GND -> +3V3
- R54 pad 2: +5V -> +3V3
- USB1 pad A6: /MCU_USB_DP -> Net-(USB1-Dp1)
- USB1 pad A7: /MCU_USB_DM -> Net-(USB1-Dn1)
- USB1 pad B6: /MCU_USB_DP -> Net-(USB1-Dp1)
- USB1 pad B7: /MCU_USB_DM -> Net-(USB1-Dn1)
Routing:
- net /MCU_RESET: track 57.8 -> 103.2 mm
- net +5V: track 325.8 -> 296.8 mm, vias 57 -> 54
- net Net-(USB1-Dp1): track 0.00 -> 16.2 mm, vias 0 -> 1
- net +3V3: track 246.9 -> 263.0 mm, vias 57 -> 59
- net Net-(USB1-Dn1): track 0.00 -> 15.9 mm, vias 0 -> 1
- net /MCU_USB_DP: track 33.9 -> 18.7 mm, vias 2 -> 1
- net /MCU_USB_DM: track 33.8 -> 18.8 mm, vias 2 -> 1
- net GND: track 89.3 -> 82.5 mm, vias 474 -> 457
- net Net-(Q2-S): track 0.00 -> 5.38 mm
- net /SWCLK: track 75.0 -> 78.7 mm
- net /SWDIO: track 73.4 -> 77.0 mm
- net Net-(Q2-G): track 14.1 -> 11.6 mm
- net Net-(U11-2Y): track 0.00 -> 1.90 mm
- net Net-(Q2-D): track 1.87 -> 0.00 mm
- net /BUS_RES/: track 35.6 -> 37.1 mm
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