File: hardware/kicad/DrunkPCDebugger.kicad_pcb (KiCad board)
At the start: 4 copper layers, 71 x 57.5 mm, 98 parts, among them Q2 AO3401A, Q3 AO3401A, Q4 AO3400A, SW2 TS3643TP, SW3 TS3643TP, U1 SN74LVC4245APWR, U10 A-SC6302R6AGHC-A03-2T, U11 SN74LVC3G07DCTR, U2 STM32H723VGT6, U3 SN74LVC4245APWR, U4 SN74LVC4245APWR, U5 X6521FV-2X27-C85D32, U6 AMS1117-3_3, U7 SN74LVC4245APWR, U8 SN74LVC3G17DCTR, X1 X322525MOB4SI

Commit message: Fix DRC
Parts:
- moved R49 4.28 mm to (89.2, 56.2), turned to 0 degrees
Routing:
- net +3V3: track 263.0 -> 274.8 mm, vias 59 -> 58
- net /SWDIO: track 77.0 -> 76.1 mm
- net /MCU_VCAP: track 34.2 -> 33.5 mm
- net GND: track 82.5 -> 81.9 mm, vias 457 -> 461

Commit message: Fixes
Parts:
- removed R29: 0603WAF1003T5E, Resistor_SMD:R_0603_1608Metric
- removed R30: 0603WAF1000T5E, Resistor_SMD:R_0603_1608Metric
- added C7: 2.2uF, Capacitor_SMD:C_0603_1608Metric, F.Cu at (115.5, 81.4)
- added Q1: AO3400A, JLCImport:AO3400A, B.Cu at (60.3, 63.9)
- added R32: 0603WAF1001T5E, Resistor_SMD:R_0603_1608Metric, F.Cu at (71.0, 53.1)
- added R33: 0603WAF1003T5E, Resistor_SMD:R_0603_1608Metric, B.Cu at (67.3, 56.6)
- added R34: 47kΩ, Resistor_SMD:R_0603_1608Metric, B.Cu at (67.3, 61.3)
- added R35: 47kΩ, Resistor_SMD:R_0603_1608Metric, F.Cu at (117.1, 81.4)
- added R57: 0603WAF1002T5E, Resistor_SMD:R_0603_1608Metric, B.Cu at (63.0, 63.9)
- added R58: 0603WAF1002T5E, Resistor_SMD:R_0603_1608Metric, F.Cu at (115.6, 77.3)
- U2: value STM32H723VGT6 -> STM32H723VET6; footprint JLCImport:STM32H723VGT6 -> JLCImport:STM32H723VET6
- moved C75 24.1 mm to (78.3, 59.5), turned to 90 degrees
Connections:
- C67 pad 1: +5V -> BUS_5V
- C69 pad 1: +5V -> BUS_5V
- C71 pad 1: +5V -> BUS_5V
- C73 pad 1: +5V -> BUS_5V
- H2 pad 1: +5V -> +3V3
- R56 pad 1: +3V3 -> BUS_5V
- R56 pad 2: /MCU_BUS_OE/ -> /BUS_OE/
- U1 pad 1: +5V -> BUS_5V
- U1 pad 22: /MCU_BUS_OE/ -> /BUS_OE/
- U2 pad 67: unconnected-(U2-PA8-Pad67) -> /MCU_BUS_5V_ADC
- U3 pad 1: +5V -> BUS_5V
- U3 pad 22: /MCU_BUS_OE/ -> /BUS_OE/
- U4 pad 1: +5V -> BUS_5V
- U4 pad 22: /MCU_BUS_OE/ -> /BUS_OE/
- U7 pad 1: +5V -> BUS_5V
- U7 pad 22: /MCU_BUS_OE/ -> /BUS_OE/
Routing:
- net +5V: track 296.8 -> 160.5 mm, vias 54 -> 50
- net BUS_5V: track 157.4 -> 285.7 mm, vias 6 -> 12
- net /MCU_BUS_OE/: track 110.1 -> 2.75 mm, vias 7 -> 0
- net /BUS_OE/: track 0.00 -> 102.6 mm, vias 0 -> 8
- net /MCU_BUS_5V_ADC: track 0.00 -> 16.1 mm, vias 0 -> 1
- net Net-(Q1-G): track 0.00 -> 15.5 mm, vias 0 -> 1
- net /MCU_VCAP: track 33.5 -> 30.0 mm
- net +3V3: track 274.8 -> 278.2 mm
- net GND: track 81.9 -> 84.7 mm, vias 461 -> 464
- net /MCU_BOOT0: track 47.9 -> 46.2 mm
- net Net-(Q2-S): track 5.38 -> 7.01 mm
- net Net-(Q2-G): track 11.6 -> 13.2 mm
- net /MCU_ADDR_BUS_DIR: track 68.4 -> 69.7 mm
- net /SWCLK: track 78.7 -> 77.7 mm
- net /MCU_RESET: track 103.2 -> 103.8 mm
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
Commit message: Pcb production
Parts:
- added R29: 10kΩ, Resistor_SMD:R_0603_1608Metric, F.Cu at (99.7, 83.5)
- added R30: 10kΩ, Resistor_SMD:R_0603_1608Metric, F.Cu at (98.9, 78.5)
- added R45: 10kΩ, Resistor_SMD:R_0603_1608Metric, F.Cu at (105.4, 85.1)
- added R46: 10kΩ, Resistor_SMD:R_0603_1608Metric, F.Cu at (105.3, 78.5)
- moved C70 0.70 mm to (105.4, 83.3)
Connections:
- U7 pad 10: unconnected-(U7-A8-Pad10) -> Net-(U7-A8)
- U7 pad 14: unconnected-(U7-B8-Pad14) -> Net-(U7-B8)
- U7 pad 21: unconnected-(U7-B1-Pad21) -> Net-(U7-B1)
- U7 pad 3: unconnected-(U7-A1-Pad3) -> Net-(U7-A1)
Routing:
- net Net-(U7-B1): track 0.00 -> 6.57 mm, vias 0 -> 1
- net Net-(U7-A1): track 0.00 -> 5.47 mm, vias 0 -> 1
- net Net-(U7-B8): track 0.00 -> 4.94 mm, vias 0 -> 1
- net Net-(U7-A8): track 0.00 -> 2.95 mm, vias 0 -> 1
- net /MCU_CTRL_BUS_DIR: track 42.6 -> 43.3 mm
- net /BUS_OE/: track 102.6 -> 103.1 mm
- net GND: track 84.7 -> 85.0 mm, vias 464 -> 466
