File: hardware/rev2/DrunkPCDebugger.kicad_pcb (KiCad board)
At the start: 4 copper layers, 71 x 57.5 mm, 94 parts, among them Q1 2N7002K-T1-GE3, Q2 AO3401A, Q3 AO3401A, SW2 TS3643TP, SW3 TS3643TP, U1 74LVX4245MTCX, U10 A-SC6302R6AGHC-A03-2T, U2 STM32H723VGT6, U3 74LVX4245MTCX, U4 74LVX4245MTCX, U5 X6521FV-2X27-C85D32, U6 AMS1117-3_3, U7 74LVX4245MTCX, U8 SN74LVC3G17DCTR, U9 SN74AHCT125DR, X1 X322525MOB4SI

Commit message: Fix errata in rev2
Parts:
- added R48: RT0603BRD0710KL, Resistor_SMD:R_0603_1608Metric, F.Cu at (53.4, 75.5)
- added R49: RT0603BRD0710KL, Resistor_SMD:R_0603_1608Metric, B.Cu at (92.2, 59.2)
- moved R47 0.16 mm to (62.6, 56.3)
Connections:
- R47 pad 2: /MCU_BUS_DIR -> /MCU_ADDR_BUS_DIR
- U1 pad 2: /MCU_BUS_DIR -> /MCU_DATA_BUS_DIR
- U2 pad 51: /MCU_BUS_DIR -> /MCU_ADDR_BUS_DIR
- U2 pad 53: unconnected-(U2-PB14-Pad53) -> /MCU_DATA_BUS_DIR
- U2 pad 9: unconnected-(U2-PC15-OSC32_OUT-Pad9) -> /MCU_CTRL_BUS_DIR
- U3 pad 2: /MCU_BUS_DIR -> /MCU_ADDR_BUS_DIR
- U4 pad 2: /MCU_BUS_DIR -> /MCU_ADDR_BUS_DIR
- U7 pad 2: /MCU_BUS_DIR -> /MCU_CTRL_BUS_DIR
Routing:
- net /MCU_BUS_DIR: track 112.0 -> 0.00 mm, vias 5 -> 0
- net /MCU_ADDR_BUS_DIR: track 0.00 -> 68.4 mm, vias 0 -> 1
- net /MCU_DATA_BUS_DIR: track 0.00 -> 46.5 mm
- net /MCU_CTRL_BUS_DIR: track 0.00 -> 33.8 mm, vias 0 -> 5
- net /MCU_BOOT0: track 56.7 -> 47.9 mm, vias 3 -> 1
- net GND: track 86.8 -> 89.0 mm, vias 473 -> 474
- net /MCU_BUS_OE/: track 108.7 -> 110.1 mm
- net /MCU_MREQ/: track 45.5 -> 44.8 mm
- net /MCU_A8: track 35.1 -> 34.6 mm
Other:
- board text added: "PCB rev 2"
