File: hardware/rev2/DrunkPCDebugger.kicad_sch (KiCad schematic)
At the start: 94 parts, among them Q1 2N7002K-T1-GE3, Q2 AO3401A, Q3 AO3401A, SW2 TS3643TP, SW3 TS3643TP, U1 74LVX4245MTCX, U10 A-SC6302R6AGHC-A03-2T, U2 STM32H723VGT6, U3 74LVX4245MTCX, U4 74LVX4245MTCX, U5 X6521FV-2X27-C85D32, U6 AMS1117-3_3, U7 74LVX4245MTCX, U8 SN74LVC3G17DCTR, U9 SN74AHCT125DR, X1 X322525MOB4SI

Commit message: Fix errata in rev2
Parts:
- added R48, R49: RT0603BRD0710KL, Resistor_SMD:R_0603_1608Metric, symbol JLCImport:RT0603BRD0710KL
Connections:
- net GND: now also R48.1, R49.1
- net MCU_DATA_BUS_DIR: now reaches U2.53 (PB14)
- net MCU_DATA_BUS_DIR: now also U1.2 (T/#R), R48.2
- net MCU_CTRL_BUS_DIR: now reaches U2.9 (PC15-OSC32_OUT)
- net MCU_CTRL_BUS_DIR: now also U7.2 (T/#R), R49.2
- net MCU_BUS_DIR renamed MCU_ADDR_BUS_DIR
- net MCU_ADDR_BUS_DIR: no longer U1.2 (T/#R), U7.2 (T/#R)
- no-connect marks 43 -> 41
